Commit message: Created rough terrain obstacle in simulation.

File: march_simulation/obstacles/rough_terrain.xacro (robot description, xacro)
@@ -1,6 +1,11 @@
 <?xml version="1.0"?>
-<robot name="stairs" xmlns:xacro="http://www.ros.org/wiki/xacro">
-    <static>true</static>
+<robot name="rough_terrrain" xmlns:xacro="http://www.ros.org/wiki/xacro">
+    <gazebo>
+        <static>true</static>
+    </gazebo>
     <!-- Sizes from the rules of the cybathlon 2020 -->
+    <xacro:property name="plate_height" default="0.022"/>
+    <xacro:property name="plate_length" default="3.88"/>
+    <xacro:property name="plate_width" default="1.95"/>
     <xacro:property name="long_block_width" default="0.04"/>
     <xacro:property name="long_block_length" default="1.15"/>
@@ -21,14 +26,14 @@
     <link name="${parent_name}"/>
     <!-- Links -->
-    <link name="step_1">
-        <collision>
-          <geometry>
-            <box size="${stairs_length} ${stairs_width} ${step_height}" />
-          </geometry>
-        </collision>
-        <visual name='visual'>
-          <geometry>
-            <box size="${stairs_length} ${stairs_width} ${step_height}" />
-          </geometry>
+    <link name="fix_plate">
+        <collision>
+            <geometry>
+                <box size="${plate_length + 2} ${plate_width + 2} ${plate_height}" />
+            </geometry>
+        </collision>
+        <visual name='visual'>
+            <geometry>
+                <box size="${plate_length + 2} ${plate_width + 2} ${plate_height}" />
+            </geometry>
         </visual>
         <inertial>
@@ -44,100 +49,356 @@
         </inertial>
     </link>
-    <link name="step_2">
-        <collision>
-          <origin xyz="0 0 0" rpy="0 0 0"/>
-          <geometry>
-            <box size="${stairs_length - 2 * step_depth} ${stairs_width} ${step_height}" />
-          </geometry>
-        </collision>
-        <visual name='visual'>
-          <origin xyz="0 0 0" rpy="0 0 0"/>
-          <geometry>
-            <box size="${stairs_length - 2 * step_depth} ${stairs_width} ${step_height}" />
-          </geometry>
-        </visual>
-    </link>
-    <link name="step_3">
-        <collision>
-          <origin xyz="0 0 0" rpy="0 0 0"/>
-          <geometry>
-            <box size="${stairs_length - 4 * step_depth} ${stairs_width} ${step_height}" />
-          </geometry>
-        </collision>
-        <visual name='visual'>
-          <origin xyz="0 0 0" rpy="0 0 0"/>
-          <geometry>
-            <box size="${stairs_length - 4 * step_depth} ${stairs_width} ${step_height}" />
-          </geometry>
-        </visual>
-    </link>
-    <link name="step_4">
-        <collision>
-          <origin xyz="0 0 0" rpy="0 0 0"/>
-          <geometry>
-            <box size="${stairs_length - 6 * step_depth} ${stairs_width} ${step_height}" />
-          </geometry>
-        </collision>
-        <visual name='visual'>
-          <origin xyz="0 0 0" rpy="0 0 0"/>
-          <geometry>
-            <box size="${stairs_length - 6 * step_depth} ${stairs_width} ${step_height}" />
-          </geometry>
-        </visual>
-    </link>
-    <link name="step_5">
-        <collision>
-          <origin xyz="0 0 0" rpy="0 0 0"/>
-          <geometry>
-            <box size="${stairs_length - 8 * step_depth} ${stairs_width} ${step_height}" />
-          </geometry>
-        </collision>
-        <visual name='visual'>
-          <origin xyz="0 0 0" rpy="0 0 0"/>
-          <geometry>
-            <box size="${stairs_length - 8 * step_depth} ${stairs_width} ${step_height}" />
-          </geometry>
-        </visual>
-    </link>
-    <link name="step_6">
-        <collision>
-          <origin xyz="0 0 0" rpy="0 0 0"/>
-          <geometry>
-            <box size="${stairs_length - 10 * step_depth} ${stairs_width} ${step_height}" />
-          </geometry>
-        </collision>
-        <visual name='visual'>
-          <origin xyz="0 0 0" rpy="0 0 0"/>
-          <geometry>
-            <box size="${stairs_length - 10 * step_depth} ${stairs_width} ${step_height}" />
-          </geometry>
-        </visual>
-    </link>
-    <gazebo reference="step_1">
-        <mu1>${mu1}</mu1>
-        <mu2>${mu2}</mu2>
-        <minDepth>${min_depth}</minDepth>
-    </gazebo>
-    <gazebo reference="step_2">
-        <mu1>${mu1}</mu1>
-        <mu2>${mu2}</mu2>
-        <minDepth>${min_depth}</minDepth>
-    </gazebo>
-    <gazebo reference="step_3">
-        <mu1>${mu1}</mu1>
-        <mu2>${mu2}</mu2>
-        <minDepth>${min_depth}</minDepth>
-    </gazebo>
-    <gazebo reference="step_4">
-        <mu1>${mu1}</mu1>
-        <mu2>${mu2}</mu2>
-        <minDepth>${min_depth}</minDepth>
-    </gazebo>
-    <gazebo reference="step_5">
-        <mu1>${mu1}</mu1>
-        <mu2>${mu2}</mu2>
-        <minDepth>${min_depth}</minDepth>
-    </gazebo>
-    <gazebo reference="step_6">
+    <link name="bottom_plate">
+        <collision>
+            <geometry>
+                <box size="${plate_length} ${plate_width} ${plate_height}" />
+            </geometry>
+        </collision>
+        <visual name='visual'>
+          <geometry>
+            <box size="${plate_length} ${plate_width} ${plate_height}" />
+          </geometry>
+        </visual>
+        <inertial>
+            <origin xyz="0 0 0" rpy="0 0 0"/>
+            <mass value="1"/>
+            <inertia
+                    ixx="1"
+                    ixy="1"
+                    ixz="1"
+                    iyy="1"
+                    iyz="1"
+                    izz="1" />
+        </inertial>
+    </link>
+    <link name="long_block_1">
+        <collision>
+          <origin xyz="0 0 0" rpy="0 0 0"/>
+          <geometry>
+            <box size="${long_block_length} ${long_block_width} ${long_block_width}" />
+          </geometry>
+        </collision>
+        <visual name='visual'>
+          <origin xyz="0 0 0" rpy="0 0 0"/>
+          <geometry>
+            <box size="${long_block_length} ${long_block_width} ${long_block_width}" />
+          </geometry>
+        </visual>
+    </link>
+    <link name="long_block_2">
+        <collision>
+            <origin xyz="0 0 0" rpy="0 0 0"/>
+            <geometry>
+                <box size="${long_block_length} ${long_block_width} ${long_block_width}" />
+            </geometry>
+        </collision>
+        <visual name='visual'>
+            <origin xyz="0 0 0" rpy="0 0 0"/>
+            <geometry>
+                <box size="${long_block_length} ${long_block_width} ${long_block_width}" />
+            </geometry>
+        </visual>
+    </link>
+    <link name="short_block_1">
+        <collision>
+          <origin xyz="0 0 0" rpy="0 0 0"/>
+          <geometry>
+            <box size="${short_block_length} ${short_block_width} ${short_block_width}" />
+          </geometry>
+        </collision>
+        <visual name='visual'>
+          <origin xyz="0 0 0" rpy="0 0 0"/>
+          <geometry>
+            <box size="${short_block_length} ${short_block_width} ${short_block_width}" />
+          </geometry>
+        </visual>
+    </link>
+    <link name="short_block_2">
+        <collision>
+            <origin xyz="0 0 0" rpy="0 0 0"/>
+            <geometry>
+                <box size="${short_block_length} ${short_block_width} ${short_block_width}" />
+            </geometry>
+        </collision>
+        <visual name='visual'>
+            <origin xyz="0 0 0" rpy="0 0 0"/>
+            <geometry>
+                <box size="${short_block_length} ${short_block_width} ${short_block_width}" />
+            </geometry>
+        </visual>
+    </link>
+    <link name="side_rod_1">
+        <collision>
+          <origin xyz="0 0 0" rpy="0 0 0"/>
+          <geometry>
+            <cylinder length="${side_rods_length}" radius="${side_rods_radius}" />
+          </geometry>
+        </collision>
+        <visual name='visual'>
+          <origin xyz="0 0 0" rpy="0 0 0"/>
+          <geometry>
+            <cylinder length="${side_rods_length}" radius="${side_rods_radius}" />
+          </geometry>
+        </visual>
+    </link>
+    <link name="side_rod_2">
+        <collision>
+            <origin xyz="0 0 0" rpy="0 0 0"/>
+            <geometry>
+                <cylinder length="${side_rods_length}" radius="${side_rods_radius}" />
+            </geometry>
+        </collision>
+        <visual name='visual'>
+            <origin xyz="0 0 0" rpy="0 0 0"/>
+            <geometry>
+                <cylinder length="${side_rods_length}" radius="${side_rods_radius}" />
+            </geometry>
+        </visual>
+    </link>
+    <link name="side_rod_3">
+        <collision>
+            <origin xyz="0 0 0" rpy="0 0 0"/>
+            <geometry>
+                <cylinder length="${side_rods_length}" radius="${side_rods_radius}" />
+            </geometry>
+        </collision>
+        <visual name='visual'>
+            <origin xyz="0 0 0" rpy="0 0 0"/>
+            <geometry>
+                <cylinder length="${side_rods_length}" radius="${side_rods_radius}" />
+            </geometry>
+        </visual>
+    </link>
+    <link name="side_rod_4">
+        <collision>
+            <origin xyz="0 0 0" rpy="0 0 0"/>
+            <geometry>
+                <cylinder length="${side_rods_length}" radius="${side_rods_radius}" />
+            </geometry>
+        </collision>
+        <visual name='visual'>
+            <origin xyz="0 0 0" rpy="0 0 0"/>
+            <geometry>
+                <cylinder length="${side_rods_length}" radius="${side_rods_radius}" />
+            </geometry>
+        </visual>
+    </link>
+    <link name="side_rod_5">
+        <collision>
+            <origin xyz="0 0 0" rpy="0 0 0"/>
+            <geometry>
+                <cylinder length="${side_rods_length}" radius="${side_rods_radius}" />
+            </geometry>
+        </collision>
+        <visual name='visual'>
+            <origin xyz="0 0 0" rpy="0 0 0"/>
+            <geometry>
+                <cylinder length="${side_rods_length}" radius="${side_rods_radius}" />
+            </geometry>
+        </visual>
+    </link>
+    <link name="side_rod_6">
+        <collision>
+            <origin xyz="0 0 0" rpy="0 0 0"/>
+            <geometry>
+                <cylinder length="${side_rods_length}" radius="${side_rods_radius}" />
+            </geometry>
+        </collision>
+        <visual name='visual'>
+            <origin xyz="0 0 0" rpy="0 0 0"/>
+            <geometry>
+                <cylinder length="${side_rods_length}" radius="${side_rods_radius}" />
+            </geometry>
+        </visual>
+    </link>
+    <link name="side_rod_7">
+        <collision>
+            <origin xyz="0 0 0" rpy="0 0 0"/>
+            <geometry>
+                <cylinder length="${side_rods_length}" radius="${side_rods_radius}" />
+            </geometry>
+        </collision>
+        <visual name='visual'>
+            <origin xyz="0 0 0" rpy="0 0 0"/>
+            <geometry>
+                <cylinder length="${side_rods_length}" radius="${side_rods_radius}" />
+            </geometry>
+        </visual>
+    </link>
+    <link name="side_rod_8">
+        <collision>
+            <origin xyz="0 0 0" rpy="0 0 0"/>
+            <geometry>
+                <cylinder length="${side_rods_length}" radius="${side_rods_radius}" />
+            </geometry>
+        </collision>
+        <visual name='visual'>
+            <origin xyz="0 0 0" rpy="0 0 0"/>
+            <geometry>
+                <cylinder length="${side_rods_length}" radius="${side_rods_radius}" />
+            </geometry>
+        </visual>
+    </link>
+    <link name="thick_rod_1">
+        <collision>
+          <origin xyz="0 0 0" rpy="0 0 0"/>
+          <geometry>
+            <cylinder length="${middle_rods_length}" radius="${thick_rod_radius}" />
+          </geometry>
+        </collision>
+        <visual name='visual'>
+          <origin xyz="0 0 0" rpy="0 0 0"/>
+          <geometry>
+              <cylinder length="${middle_rods_length}" radius="${thick_rod_radius}" />
+          </geometry>
+        </visual>
+    </link>
+    <link name="thick_rod_2">
+        <collision>
+            <origin xyz="0 0 0" rpy="0 0 0"/>
+            <geometry>
+                <cylinder length="${middle_rods_length}" radius="${thick_rod_radius}" />
+            </geometry>
+        </collision>
+        <visual name='visual'>
+            <origin xyz="0 0 0" rpy="0 0 0"/>
+            <geometry>
+                <cylinder length="${middle_rods_length}" radius="${thick_rod_radius}" />
+            </geometry>
+        </visual>
+    </link>
+    <link name="thick_rod_3">
+        <collision>
+            <origin xyz="0 0 0" rpy="0 0 0"/>
+            <geometry>
+                <cylinder length="${middle_rods_length}" radius="${thick_rod_radius}" />
+            </geometry>
+        </collision>
+        <visual name='visual'>
+            <origin xyz="0 0 0" rpy="0 0 0"/>
+            <geometry>
+                <cylinder length="${middle_rods_length}" radius="${thick_rod_radius}" />
+            </geometry>
+        </visual>
+    </link>
+    <link name="thin_rod_1">
+        <collision>
+          <origin xyz="0 0 0" rpy="0 0 0"/>
+          <geometry>
+              <cylinder length="${middle_rods_length}" radius="${thin_rod_radius}" />
+          </geometry>
+        </collision>
+        <visual name='visual'>
+          <origin xyz="0 0 0" rpy="0 0 0"/>
+          <geometry>
+              <cylinder length="${middle_rods_length}" radius="${thin_rod_radius}" />
+          </geometry>
+        </visual>
+    </link>
+    <link name="thin_rod_2">
+        <collision>
+            <origin xyz="0 0 0" rpy="0 0 0"/>
+            <geometry>
+                <cylinder length="${middle_rods_length}" radius="${thin_rod_radius}" />
+            </geometry>
+        </collision>
+        <visual name='visual'>
+            <origin xyz="0 0 0" rpy="0 0 0"/>
+            <geometry>
+                <cylinder length="${middle_rods_length}" radius="${thin_rod_radius}" />
+            </geometry>
+        </visual>
+    </link>
+    <gazebo reference="bottom_plate">
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
Commit message: Removed the fix plate under the rough terrain.

File: march_simulation/obstacles/rough_terrain.xacro (robot description, xacro)
@@ -26,14 +26,37 @@
     <link name="${parent_name}"/>
     <!-- Links -->
-    <link name="fix_plate">
-        <collision>
-            <geometry>
-                <box size="${plate_length + 2} ${plate_width + 2} ${plate_height}" />
-            </geometry>
-        </collision>
-        <visual name='visual'>
-            <geometry>
-                <box size="${plate_length + 2} ${plate_width + 2} ${plate_height}" />
-            </geometry>
+<!--    <link name="fix_plate">-->
+<!--        <collision>-->
+<!--            <geometry>-->
+<!--                <box size="${plate_length + 2} ${plate_width + 2} ${plate_height}" />-->
+<!--            </geometry>-->
+<!--        </collision>-->
+<!--        <visual name='visual'>-->
+<!--            <geometry>-->
+<!--                <box size="${plate_length + 2} ${plate_width + 2} ${plate_height}" />-->
+<!--            </geometry>-->
+<!--        </visual>-->
+<!--        <inertial>-->
+<!--            <origin xyz="0 0 0" rpy="0 0 0"/>-->
+<!--            <mass value="1"/>-->
+<!--            <inertia-->
+<!--                    ixx="1"-->
+<!--                    ixy="1"-->
+<!--                    ixz="1"-->
+<!--                    iyy="1"-->
+<!--                    iyz="1"-->
+<!--                    izz="1" />-->
+<!--        </inertial>-->
+<!--    </link>-->
+    <link name="bottom_plate">
+        <collision>
+            <geometry>
+                <box size="${plate_length} ${plate_width} ${plate_height}" />
+            </geometry>
+        </collision>
+        <visual name='visual'>
+          <geometry>
+            <box size="${plate_length} ${plate_width} ${plate_height}" />
+          </geometry>
         </visual>
         <inertial>
@@ -49,27 +72,4 @@
         </inertial>
     </link>
-    <link name="bottom_plate">
-        <collision>
-            <geometry>
-                <box size="${plate_length} ${plate_width} ${plate_height}" />
-            </geometry>
-        </collision>
-        <visual name='visual'>
-          <geometry>
-            <box size="${plate_length} ${plate_width} ${plate_height}" />
-          </geometry>
-        </visual>
-        <inertial>
-            <origin xyz="0 0 0" rpy="0 0 0"/>
-            <mass value="1"/>
-            <inertia
-                    ixx="1"
-                    ixy="1"
-                    ixz="1"
-                    iyy="1"
-                    iyz="1"
-                    izz="1" />
-        </inertial>
-    </link>
     <link name="long_block_1">
         <collision>
@@ -315,9 +315,9 @@
         <minDepth>${min_depth}</minDepth>
     </gazebo>
-    <gazebo reference="fix_plate">
-        <mu1>${mu1}</mu1>
-        <mu2>${mu2}</mu2>
-        <minDepth>${min_depth}</minDepth>
-    </gazebo>
+<!--    <gazebo reference="fix_plate">-->
+<!--        <mu1>${mu1}</mu1>-->
+<!--        <mu2>${mu2}</mu2>-->
+<!--        <minDepth>${min_depth}</minDepth>-->
+<!--    </gazebo>-->
     <gazebo reference="long_block_1">
         <mu1>${mu1}</mu1>
@@ -406,13 +406,13 @@
     </gazebo>
     <!-- Joints -->
-    <joint name="joint_fix" type="fixed">
+<!--    <joint name="joint_fix" type="fixed">-->
+<!--        <parent link="${parent_name}"/>-->
+<!--        <child link="fix_plate"/>-->
+<!--        <origin xyz="${- plate_length} 0 ${plate_height}" rpy="0 0 0"/>-->
+<!--    </joint>-->
+    <joint name="joint_0" type="fixed">
         <parent link="${parent_name}"/>
-        <child link="fix_plate"/>
-        <origin xyz="${- plate_length} 0 ${plate_height}" rpy="0 0 0"/>
-    </joint>
-    <joint name="joint_0" type="fixed">
-        <parent link="fix_plate"/>
         <child link="bottom_plate"/>
-        <origin xyz="0 0 ${plate_height}" rpy="0 0 0"/>
+        <origin xyz="-2.5  0 ${plate_height}" rpy="0 0 0"/>
     </joint>
     <joint name="joint_1" type="fixed">

Commit message: Deleted the fix plate code (was already in comment)

File: march_simulation/obstacles/rough_terrain.xacro (robot description, xacro)
@@ -25,28 +25,4 @@
     <!-- Used for fixing robot to Gazebo 'base_link' -->
     <link name="${parent_name}"/>
-    <!-- Links -->
-<!--    <link name="fix_plate">-->
-<!--        <collision>-->
-<!--            <geometry>-->
-<!--                <box size="${plate_length + 2} ${plate_width + 2} ${plate_height}" />-->
-<!--            </geometry>-->
-<!--        </collision>-->
-<!--        <visual name='visual'>-->
-<!--            <geometry>-->
-<!--                <box size="${plate_length + 2} ${plate_width + 2} ${plate_height}" />-->
-<!--            </geometry>-->
-<!--        </visual>-->
-<!--        <inertial>-->
-<!--            <origin xyz="0 0 0" rpy="0 0 0"/>-->
-<!--            <mass value="1"/>-->
-<!--            <inertia-->
-<!--                    ixx="1"-->
-<!--                    ixy="1"-->
-<!--                    ixz="1"-->
-<!--                    iyy="1"-->
-<!--                    iyz="1"-->
-<!--                    izz="1" />-->
-<!--        </inertial>-->
-<!--    </link>-->
     <link name="bottom_plate">
         <collision>
@@ -315,9 +291,4 @@
         <minDepth>${min_depth}</minDepth>
     </gazebo>
-<!--    <gazebo reference="fix_plate">-->
-<!--        <mu1>${mu1}</mu1>-->
-<!--        <mu2>${mu2}</mu2>-->
-<!--        <minDepth>${min_depth}</minDepth>-->
-<!--    </gazebo>-->
     <gazebo reference="long_block_1">
         <mu1>${mu1}</mu1>
@@ -406,9 +377,4 @@
     </gazebo>
     <!-- Joints -->
-<!--    <joint name="joint_fix" type="fixed">-->
-<!--        <parent link="${parent_name}"/>-->
-<!--        <child link="fix_plate"/>-->
-<!--        <origin xyz="${- plate_length} 0 ${plate_height}" rpy="0 0 0"/>-->
-<!--    </joint>-->
     <joint name="joint_0" type="fixed">
         <parent link="${parent_name}"/>
