Commit message: Made the right shape of the tilted path

File: march_simulation/obstacles/tilted_path.xacro (robot description, xacro)
@@ -4,8 +4,8 @@
     <!-- Sizes from the rules of the cybathlon 2020 -->
     <xacro:property name="middle_block_length" default="3"/>
-    <xacro:property name="middle_block_width" default="1.5"/>
+    <xacro:property name="middle_block_width" default="1.474"/>
     <xacro:property name="middle_block_height" default="0.5"/>
     <xacro:property name="middle_block_angle" default="0.21"/>
-    <xacro:property name="side_blocks_length" default="1.5"/>
+    <xacro:property name="side_blocks_length" default="1.474"/>
     <xacro:property name="side_blocks_width" default="1.5"/>
     <xacro:property name="side_blocks_height" default="0.5"/>
@@ -90,15 +90,15 @@
         <parent link="${parent_name}"/>
         <child link="middle_block"/>
-        <origin xyz="${-distance_to_origin} 0 0" rpy="${- middle_block_angle} 0 0"/>
+        <origin xyz="${-distance_to_origin-2.5} 0 -0.15" rpy="${- middle_block_angle} 0 0"/>
     </joint>
     <joint name="joint_1" type="fixed">
         <parent link="middle_block"/>
         <child link="side_block_1"/>
-        <origin xyz="2.1 0 -0.2" rpy="${- middle_block_angle} ${side_blocks_angle} 0"/>
+        <origin xyz="2.17 0.01 -0.135" rpy="0 ${side_blocks_angle} 0"/>
     </joint>
     <joint name="joint_2" type="fixed">
         <parent link="middle_block"/>
         <child link="side_block_2"/>
-        <origin xyz="-2.1 0 -0.2" rpy="${- middle_block_angle} ${-side_blocks_angle} 0"/>
+        <origin xyz="-2.17 0.01 -0.135" rpy="0 ${-side_blocks_angle} 0"/>
     </joint>
 </robot>

Commit message: Renamed joint names

File: march_simulation/obstacles/tilted_path.xacro (robot description, xacro)
@@ -89,15 +89,15 @@
     </gazebo>
     <!-- Joints -->
-    <joint name="hip" type="fixed">
+    <joint name="joint_1" type="fixed">
         <parent link="${parent_name}"/>
         <child link="middle_block"/>
         <origin xyz="${-distance_to_origin-2.5} 0 -0.15" rpy="${- middle_block_angle} 0 0"/>
     </joint>
-    <joint name="joint_1" type="fixed">
+    <joint name="joint_2" type="fixed">
         <parent link="middle_block"/>
         <child link="side_block_1"/>
         <origin xyz="2.17 0.01 -0.135" rpy="0 ${side_blocks_angle} 0"/>
     </joint>
-    <joint name="joint_2" type="fixed">
+    <joint name="joint_3" type="fixed">
         <parent link="middle_block"/>
         <child link="side_block_2"/>
